Commit message: state manager&camera added (not working properly)

File: exp_assignment2/urdf/robot.xacro (robot description, xacro)
@@ -185,5 +185,5 @@
 	    <inertial>
 	      <mass value="1e-5" />
-	      <origin xyz="0 0 0.23" rpy="0 0 0"/>
+	      <origin xyz="0 0 0" rpy="0 0 0"/>
 	      <inertia ixx="1e-6" ixy="0" ixz="0" iyy="1e-6" iyz="0" izz="1e-6" />
 	    </inertial>
@@ -195,5 +195,5 @@
 	    <child link="camera_link"/>
 	 </joint>
-<transmission name="head_hoint_trans">
+<transmission name="head_joint_trans">
 	<type>transmission_interface/SimpleTransmission</type>
 	<joint name="head_joint">

Commit message: Controller updatated

File: exp_assignment2/urdf/robot.xacro (robot description, xacro)
@@ -1,44 +1,45 @@
 <?xml version="1.0"?>
 <robot xmlns:xacro="http://www.ros.org/wiki/xacro" name="robot_xacro">
-<xacro:include filename="$(find exp_assignment2)/urdf/robot.gazebo"/>
-	<xacro:property name="length_wheel" value="0.04" />
-	<xacro:property name="radius_wheel" value="0.1" />
-	<xacro:macro name="default_inertial" params="mass">
-               <inertial>
-                       <mass value="${mass}" />
-                       <origin rpy="0 1.5707 1.5707" xyz="0 0 0"/>
-                       <inertia ixx="0.000526666666667" ixy="0" ixz="0" iyy="0.000526666666667" iyz="0" izz="0.001"/>
-               </inertial>
+	<xacro:include filename="$(find exp_assignment2)/urdf/robot.gazebo"/>
+		<xacro:property name="length_wheel" value="0.04" />
+		<xacro:property name="radius_wheel" value="0.1" />
+		<xacro:macro name="default_inertial" params="mass">
+		       <inertial>
+		       <mass value="${mass}" />
+		       <origin rpy="0 1.5707 1.5707" xyz="0 0 0"/>
+		       <inertia ixx="0.000526666666667" ixy="0" ixz="0" iyy="0.000526666666667" iyz="0" izz="0.001"/>
+		       </inertial>
+		</xacro:macro>
+		<xacro:macro name="wheel_geometry">
+		<geometry>
+			<cylinder length="${length_wheel}" radius="${radius_wheel}"/>
+		</geometry>
 	</xacro:macro>
-    <xacro:macro name="wheel_geometry">
-		<geometry>
-       			<cylinder length="${length_wheel}" radius="${radius_wheel}"/>
-     	</geometry>
-	</xacro:macro>
-  <material name="black">
-    <color rgba="0.0 0.0 0.0 1.0"/>
-  </material>
-  <material name="blue">
-    <color rgba="0.203125 0.23828125 0.28515625 1.0"/>
-  </material>
-  <material name="green">
-    <color rgba="0.0 0.8 0.0 1.0"/>
-  </material>
-  <material name="grey">
-    <color rgba="0.2 0.2 0.2 1.0"/>
-  </material>
-  <material name="orange">
-    <color rgba="1.0 0.423529411765 0.0392156862745 1.0"/>
-  </material>
-  <material name="brown">
-    <color rgba="0.870588235294 0.811764705882 0.764705882353 1.0"/>
-  </material>
-  <material name="red">
-    <color rgba="0.80078125 0.12890625 0.1328125 1.0"/>
-  </material>
-  <material name="white">
-    <color rgba="1.0 1.0 1.0 1.0"/>
-  </material>
-	  <link name="link_chassis">
+	<material name="black">
+		<color rgba="0.0 0.0 0.0 1.0"/>
+	</material>
+	<material name="blue">
+		<color rgba="0.203125 0.23828125 0.28515625 1.0"/>
+	</material>
+	<material name="green">
+		<color rgba="0.0 0.8 0.0 1.0"/>
+	</material>
+	<material name="grey">
+		<color rgba="0.2 0.2 0.2 1.0"/>
+	</material>
+	<material name="orange">
+		<color rgba="1.0 0.423529411765 0.0392156862745 1.0"/>
+	</material>
+	<material name="brown">
+		<color rgba="0.870588235294 0.811764705882 0.764705882353 1.0"/>
+	</material>
+	<material name="red">
+		<color rgba="0.80078125 0.12890625 0.1328125 1.0"/>
+	</material>
+	<material name="white">
+		<color rgba="1.0 1.0 1.0 1.0"/>
+	</material>
+<!--************************************LINKS****************************************-->
+<link name="link_chassis">
     <!-- pose and inertial -->
     <pose>0 0 0.1 0 0 0</pose>
@@ -77,7 +78,7 @@
   <link name="neck_link">
   	<inertial>
-  		<mass value="0.025"/>
-  		<origin xyz="0 0 0" rpy="0.05 0 0" />
-  		<inertia ixx="0.000010279" ixy="0" ixz="0" iyy="0.000010279" iyz="0" izz="0.000007225"/>
+	<mass value="0.025"/>
+	<origin xyz="0 0 0" rpy="0.05 0 0" />
+	<inertia ixx="0.000010279" ixy="0" ixz="0" iyy="0.000010279" iyz="0" izz="0.000007225"/>
   	</inertial>
   	<collision>
@@ -95,14 +96,9 @@
   	</visual>
   </link>
-  <joint name="base_to_neck" type="fixed">
-  	<origin rpy="0 0 0" xyz="0.26 0 0"/> <!--0.06-->
-  	<parent link="link_chassis"/>
-  	<child link="neck_link"/>
-  </joint>
   <link name="head_link">
   	<inertial>
-  		<mass value="0.025"/>
-  		<origin xyz="0 0 0.18" rpy="0 0 0" />
-  		<inertia ixx="0.000010279" ixy="0" ixz="0" iyy="0.000010279" iyz="0" izz="0.000007225"/>
+	<mass value="0.025"/>
+	<origin xyz="0 0 0.18" rpy="0 0 0" />
+	<inertia ixx="0.000010279" ixy="0" ixz="0" iyy="0.000010279" iyz="0" izz="0.000007225"/>
   	</inertial>
   	<collision>
@@ -120,4 +116,51 @@
   	</visual>
   </link>
+   <link name="link_right_wheel">
+    <xacro:default_inertial mass="0.2"/>
+    <collision name="link_right_wheel_collision">
+      <origin rpy="0 1.5707 1.5707" xyz="0 0 0"/>
+      <xacro:wheel_geometry />
+    </collision>
+    <visual name="link_right_wheel_visual">
+      <origin rpy="0 1.5707 1.5707" xyz="0 0 0"/>
+      <xacro:wheel_geometry />
+      <material name="red"/>
+    </visual>
+  </link>
+   <link name="link_left_wheel">
+    <xacro:default_inertial mass="0.2"/>
+    <collision name="link_left_wheel_collision">
+      <origin rpy="0 1.5707 1.5707" xyz="0 0 0"/>
+      <xacro:wheel_geometry />
+    </collision>
+    <visual name="link_left_wheel_visual">
+      <origin rpy="0 1.5707 1.5707" xyz="0 0 0"/>
+      <xacro:wheel_geometry />
+      <material name="red"/>
+    </visual>
+  </link>
+  <link name="camera_link">
+    <collision>
+      <origin xyz="0 0 0.23" rpy="0 0 0"/>
+      <geometry>
+	<box size="0.05 0.05 0.05"/>
+      </geometry>
+    </collision>
+    <visual>
+      <origin xyz="0 0 0.23" rpy="0 0 0"/>
+      <geometry>
+	<box size="0.05 0.05 0.05"/>
+      </geometry>
+      <material name="white">
+	<color rgba="1 0 0 1"/>
+      </material>
+    </visual>
+    <inertial>
+      <mass value="1e-5" />
+      <origin xyz="0 0 0" rpy="0 0 0"/>
+      <inertia ixx="1e-6" ixy="0" ixz="0" iyy="1e-6" iyz="0" izz="1e-6" />
+    </inertial>
+  </link>
+<!--************************************JOINTS****************************************-->
   <joint name="head_joint" type="revolute">
   	<axis xyz="0 0 1"/>
@@ -127,28 +170,4 @@
   	<child link="head_link"/>
   </joint>
-   <link name="link_right_wheel">
-    <xacro:default_inertial mass="0.2"/>
-    <collision name="link_right_wheel_collision">
-      <origin rpy="0 1.5707 1.5707" xyz="0 0 0"/>
-      <xacro:wheel_geometry />
-    </collision>
-    <visual name="link_right_wheel_visual">
-      <origin rpy="0 1.5707 1.5707" xyz="0 0 0"/>
-      <xacro:wheel_geometry />
-      <material name="red"/>
-    </visual>
-  </link>
-   <link name="link_left_wheel">
-    <xacro:default_inertial mass="0.2"/>
-    <collision name="link_left_wheel_collision">
-      <origin rpy="0 1.5707 1.5707" xyz="0 0 0"/>
-      <xacro:wheel_geometry />
-    </collision>
-    <visual name="link_left_wheel_visual">
-      <origin rpy="0 1.5707 1.5707" xyz="0 0 0"/>
-      <xacro:wheel_geometry />
-      <material name="red"/>
-    </visual>
-  </link>
   <joint name="joint_right_wheel" type="continuous">
     <origin rpy="0 0 0" xyz="-0.05 0.15 0"/>
@@ -167,32 +186,16 @@
     <joint_properties damping="1.0" friction="1.0"/>
   </joint>
-  <link name="camera_link">
-	    <collision>
-	      <origin xyz="0 0 0.23" rpy="0 0 0"/>
-	      <geometry>
-		<box size="0.05 0.05 0.05"/>
-	      </geometry>
-	    </collision>
-	    <visual>
-	      <origin xyz="0 0 0.23" rpy="0 0 0"/>
-	      <geometry>
-		<box size="0.05 0.05 0.05"/>
-	      </geometry>
-	      <material name="white">
-		<color rgba="1 0 0 1"/>
-	      </material>
-	    </visual>
-	    <inertial>
-	      <mass value="1e-5" />
-	      <origin xyz="0 0 0" rpy="0 0 0"/>
-	      <inertia ixx="1e-6" ixy="0" ixz="0" iyy="1e-6" iyz="0" izz="1e-6" />
-	    </inertial>
-  </link>
+  <joint name="base_to_neck" type="fixed">
+  	<origin rpy="0 0 0" xyz="0.26 0 0"/> <!--0.06-->
+  	<parent link="link_chassis"/>
+  	<child link="neck_link"/>
+  </joint>
   <joint name="camera_joint" type="fixed">
-	    <axis xyz="0 1 0" />
+	    <axis xyz="1 0 0" />
 	    <origin xyz="0 0 0" rpy="0 0 0"/>
 	    <parent link="head_link"/>
 	    <child link="camera_link"/>
-	 </joint>
+  </joint>
+<!--************************************TRANSMISSION****************************************-->
 <transmission name="head_joint_trans">
 	<type>transmission_interface/SimpleTransmission</type>
